File: WiREDSchema.brd (EAGLE design)
At the start: 33.3 x 28.6 mm, 27 parts, among them U1 MCP73831, U2 TPS61200, X1 USB-MICROB

Commit message: Gerber and shift down
Parts:
- moved U1 0.63 mm to (11.4, 14.0)
Routing:
- net VBATT: track 70.8 -> 71.8 mm
- net N$14: track 10.4 -> 11.1 mm
- net N$11: track 12.1 -> 12.7 mm
- net 5VIN: track 39.0 -> 39.6 mm
Changed lines of the file:
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@@
 <attribute name="OC_FARNELL" value="2331533" x="33.655" y="-10.16" size="1.778" layer="27" display="off"/>
 </element>
-<element name="U1" library="SparkFun" package="SOT23-5" value="MCP73831" x="11.43" y="14.605">
-<attribute name="MPN" value="MCP73831T-2ACI/OT" x="26.67" y="-5.715" size="1.778" layer="27" display="off"/>
-<attribute name="MF" value="MICROCHIP" x="26.67" y="-5.715" size="1.778" layer="27" display="off"/>
-<attribute name="OC_FARNELL" value="1332158" x="26.67" y="-5.715" size="1.778" layer="27" display="off"/>
+<element name="U1" library="SparkFun" package="SOT23-5" value="MCP73831" x="11.43" y="13.97">
+<attribute name="MPN" value="MCP73831T-2ACI/OT" x="26.67" y="-6.35" size="1.778" layer="27" display="off"/>
+<attribute name="MF" value="MICROCHIP" x="26.67" y="-6.35" size="1.778" layer="27" display="off"/>
+<attribute name="OC_FARNELL" value="1332158" x="26.67" y="-6.35" size="1.778" layer="27" display="off"/>
 </element>
 <element name="R5" library="SparkFun" package="0402-RES" value="2k" x="15.875" y="25.4">
@@
 <contactref element="C6" pad="2"/>
 <contactref element="JP3" pad="2"/>
-<wire x1="11.43" y1="13.3049" x2="11.43" y2="20.32" width="0.254" layer="1"/>
+<wire x1="11.43" y1="12.6699" x2="11.43" y2="20.32" width="0.254" layer="1"/>
 <wire x1="11.43" y1="20.32" x2="11.445" y2="20.32" width="0.254" layer="1"/>
 <wire x1="8.89" y1="18.796" x2="7.366" y2="20.32" width="0.254" layer="1"/>
@@
 <wire x1="10.16" y1="12.192" x2="8.89" y2="13.462" width="0.254" layer="1"/>
 <wire x1="11.43" y1="12.192" x2="10.16" y2="12.192" width="0.254" layer="1"/>
-<wire x1="11.43" y1="13.3049" x2="11.43" y2="12.192" width="0.254" layer="1"/>
+<wire x1="11.43" y1="12.6699" x2="11.43" y2="12.192" width="0.254" layer="1"/>
 <wire x1="7.366" y1="20.32" x2="7.27" y2="20.36" width="0.254" layer="1"/>
 <wire x1="8.89" y1="5.08" x2="7.112" y2="5.08" width="0.254" layer="1"/>
@@
 <wire x1="12.192" y1="21.336" x2="12.192" y2="24.892" width="0.254" layer="1"/>
 <wire x1="11.684" y1="25.4" x2="11.545" y2="25.4" width="0.254" layer="1"/>
-<wire x1="12.192" y1="16.002" x2="12.38" y2="15.9051" width="0.254" layer="1"/>
+<wire x1="12.192" y1="16.002" x2="12.38" y2="15.2701" width="0.254" layer="1"/>
 <wire x1="11.176" y1="21.336" x2="10.16" y2="20.32" width="0.254" layer="1"/>
 <wire x1="12.192" y1="21.336" x2="11.176" y2="21.336" width="0.254" layer="1"/>
@@
 <wire x1="12.954" y1="12.7" x2="12.446" y2="13.208" width="0.254" layer="1"/>
 <wire x1="12.954" y1="8.382" x2="12.954" y2="12.7" width="0.254" layer="1"/>
-<wire x1="12.446" y1="13.208" x2="12.38" y2="13.3049" width="0.254" layer="1"/>
+<wire x1="12.446" y1="13.208" x2="12.38" y2="12.6699" width="0.254" layer="1"/>
 <wire x1="12.954" y1="8.382" x2="12.97" y2="8.145" width="0.254" layer="1"/>
 <wire x1="13.208" y1="16.002" x2="14.986" y2="17.78" width="0.254" layer="1"/>
@@
 <wire x1="12.446" y1="13.462" x2="13.208" y2="14.224" width="0.254" layer="1"/>
 <wire x1="14.986" y1="17.78" x2="15.225" y2="17.78" width="0.254" layer="1"/>
-<wire x1="12.446" y1="13.462" x2="12.38" y2="13.3049" width="0.254" layer="1"/>
+<wire x1="12.446" y1="13.462" x2="12.38" y2="12.6699" width="0.254" layer="1"/>
 <wire x1="20.32" y1="17.78" x2="20.32" y2="14.224" width="0.254" layer="1"/>
 <wire x1="20.32" y1="14.224" x2="20.32" y2="13.716" width="0.254" layer="1"/>
@@
 <wire x1="10.414" y1="16.002" x2="10.414" y2="17.272" width="0.254" layer="1"/>
 <wire x1="14.986" y1="25.4" x2="15.225" y2="25.4" width="0.254" layer="1"/>
-<wire x1="10.414" y1="16.002" x2="10.48" y2="15.9051" width="0.254" layer="1"/>
+<wire x1="10.414" y1="16.002" x2="10.48" y2="15.2701" width="0.254" layer="1"/>
 <via x="13.208" y="19.304" extent="1-16" drill="0.6096"/>
 <via x="10.414" y="17.272" extent="1-16" drill="0.6096"/>
@@
 <wire x1="10.414" y1="13.462" x2="9.398" y2="14.478" width="0.254" layer="1"/>
 <wire x1="9.906" y1="22.86" x2="10.145" y2="22.86" width="0.254" layer="1"/>
-<wire x1="10.414" y1="13.462" x2="10.48" y2="13.3049" width="0.254" layer="1"/>
+<wire x1="10.414" y1="13.462" x2="10.48" y2="12.6699" width="0.254" layer="1"/>
 </signal>
 <signal name="N$8">
